Commit message: Add files via upload

File: src/robot_description/urdf/schunk_egh80/schunk_egh80_gripper.transmission.xacro (robot description, xacro)
@@ -2,4 +2,14 @@
 <robot xmlns:xacro="http://www.ros.org/wiki/xacro">
   <xacro:macro name="schunk_egh80_gripper_transmission" params="prefix">
+    <transmission name="${prefix}dedo_dir_joint_trans"/>
+      <type>transmission_interface/SimpleTransmission</type>
+      <joint name="${prefix}dedo_dir_joint">
+        <hardwareInterface>PositionJointInterface</hardwareInterface>
+      </joint>
+      <actuator name="${prefix}dedo_dir_joint_motor">
+        <mechanicalReduction>1</mechanicalReduction>
+        <motorTorqueConstant>1</motorTorqueConstant>
+      </actuator>
+    </transmission>
     <transmission name="${prefix}dedo_esq_joint_trans"/>
       <type>transmission_interface/SimpleTransmission</type>

File: src/robot_description/urdf/schunk_egh80/schunk_egh80_gripper.urdf.xacro (robot description, xacro)
@@ -5,23 +5,7 @@
         <!-- Gripper-->
         <link name="schunk_egh80_link">
-            <!--<visual>
-                <origin xyz="0.0 0.001000000000000025608 0.0" rpy="2.9837243786801082024e-16 -0 0" />
-                <geometry>
-                    <xacro:get_mesh name="gripper_connector" type="visual"/>
-                </geometry>
-                <material name="conector_tcp_material">
-                    <color rgba="0.50196078431372548323 0.50196078431372548323 0.50196078431372548323 1.0"/>
-                </material>
-            </visual>
-            <collision>
-                <origin xyz="0.0 0.001000000000000025608 -3.8353651851674719353e-17" rpy="2.9837243786801082024e-16 -0 0" />
-                <geometry>
-                    <xacro:get_mesh name="gripper_connector" type="collision"/>
-                </geometry>
-            </collision> -->
             <visual>
                 <origin xyz="0.0 0.036423269171482079709 0.075503655548620457472" rpy="-1.3439035240356334011 -0 0" />
                 <geometry>
-                    <!--mesh filename="etiqueta" type="visual"/-->
                     <mesh filename="package://robot_description/meshes/schunk_egh80/visual/etiqueta.dae"/>
                 </geometry>
@@ -33,6 +17,5 @@
                 <origin xyz="0.0 0.036423269171482079709 0.075503655548620457472" rpy="-1.3439035240356334011 -0 0" />
                 <geometry>
-                    <!--xacro:get_mesh filename="etiqueta" type="collision"/-->
-                    <mesh filename="package://robot_description/meshes/schunk_egh80/collision/etiqueta.stl "/>
+                    <mesh filename="package://robot_description/meshes/schunk_egh80/collision/etiqueta.stl"/>
                 </geometry>
             </collision>
@@ -40,5 +23,4 @@
                 <origin xyz="0.0 0.001000000000000025608 -3.8353651851674719353e-17" rpy="2.9837243786801082024e-16 -0 0" />
                 <geometry>
-                    <!--xacro:get_mesh filename="egh80" type="visual"/-->
                     <mesh filename="package://robot_description/meshes/schunk_egh80/visual/egh_80.dae" />
                 </geometry>
@@ -50,5 +32,4 @@
                 <origin xyz="0.0 0.001000000000000025608 -3.8353651851674719353e-17" rpy="2.9837243786801082024e-16 -0 0" />
                 <geometry>
-                    <!--xacro:get_mesh filename="egh80" type="collision"/-->
                     <mesh filename="package://robot_description/meshes/schunk_egh80/collision/egh_80.stl" />
                 </geometry>
@@ -65,6 +46,5 @@
                 <origin xyz="0.0023249999999999781258 0.08007769391666488823 0.031950000000000013112" rpy="3.141592653589793116 0 -3.141592653589793116" />
                 <geometry>
-                    <mesh filename="package://robot_description/meshes/shunk/visual/almofada.dae"/-->
-                    <!--xacro:get_mesh name="almofada" type="visual"/-->
+                    <mesh filename="package://robot_description/meshes/schunk_egh80/visual/almofada.dae"/>
                 </geometry>
             </visual>
@@ -73,5 +53,4 @@
                 <geometry>
                     <mesh filename="package://robot_description/meshes/schunk_egh80/collision/almofada.stl"/>
-                    <!--xacro:get_mesh name="almofada" type="collision"/-->
                 </geometry>
             </collision>
@@ -79,6 +58,5 @@
                 <origin xyz="0.0018250000000000375297 0.033299999999999774225 0.040700000000000007006" rpy="-9.244463733061490901e-33 1.570796326794896558 0" />
                 <geometry>
-                    <mesh filename="package://robot_description/meshes/shunk/visual/falanginha.dae"/>
-                <!--xacro:get_mesh name="falanginha" type="visual"/-->
+                    <mesh filename="package://robot_description/meshes/schunk_egh80/visual/falanginha.dae"/>
                 </geometry>
                 <material name="falanginha_material">
@@ -90,5 +68,4 @@
                 <geometry>
                     <mesh filename="package://robot_description/meshes/schunk_egh80/collision/falanginha.stl"/>
-                    <!--xacro:get_mesh name="falanginha" type="collision"/-->
                 </geometry>
             </collision>
@@ -96,6 +73,5 @@
                 <origin xyz="0.0026249999999999433509 0.033299999999999801981 0.040700000000000007006" rpy="-9.244463733061490901e-33 1.570796326794896336 0" />
                 <geometry>
-                    <mesh filename="$package://robot_description/meshes/shunk/visual/falange.dae"/>
-                    <!--xacro:get_mesh name="falange" type="visual"/-->
+                    <mesh filename="package://robot_description/meshes/schunk_egh80/visual/falange.dae"/>
                 </geometry>
                 <material name="falange_material">
@@ -107,5 +83,4 @@
                 <geometry>
                     <mesh filename="package://robot_description/meshes/schunk_egh80/collision/falange.stl"/>
-                    <!--xacro:get_mesh name="falange" type="collision"/-->
                 </geometry>
             </collision>
@@ -113,6 +88,5 @@
                 <origin xyz="0.0023249999999999772585 0.065299999999999774891 0.040700000000000007006" rpy="-9.244463733061490901e-33 1.570796326794896558 0" />
                 <geometry>
-                    <mesh filename="package://robot_description/meshes/shunk/visual/falangeta.dae"/>
-                    <!--xacro:get_mesh name="falangeta" type="visual"/-->
+                    <mesh filename="package://robot_description/meshes/schunk_egh80/visual/falangeta.dae"/>
                 </geometry>
                 <material name="falangeta_material">
@@ -124,5 +98,4 @@
                 <geometry>
                     <mesh filename="package://robot_description/meshes/schunk_egh80/collision/falangeta.stl"/>
-                    <!--xacro:get_mesh name="falangeta" type="collision" /-->
                 </geometry>
             </collision>
@@ -130,6 +103,5 @@
                 <origin xyz="0.0026250000000000014641 0.016000000000000014211 0.041500000000000009104" rpy="-9.244463733061490901e-33 1.570796326794896558 0" />
                 <geometry>
-                    <mesh filename="package://robot_description/meshes/shunk/visual/guia_dedo.dae"/>
-                    <!--xacro:get_mesh name="guia_dedo" type="visual"/-->
+                    <mesh filename="package://robot_description/meshes/schunk_egh80/visual/guia_dedo.dae"/>
                 </geometry>
                 <material name="guia_dedo_material">
@@ -140,6 +112,5 @@
                 <origin xyz="0.0026250000000000014641 0.016000000000000014211 0.041500000000000009104" rpy="-9.244463733061490901e-33 1.570796326794896558 0" />
                 <geometry>
-                    <mesh filename="package://robot_description/meshes/shunk/collision/guia_dedo.stl"/>
-                    <!--xacro:get_mesh name="guia_dedo" type="collision"/-->
+                    <mesh filename="package://robot_description/meshes/schunk_egh80/collision/guia_dedo.stl"/>
                 </geometry>
             </collision>
@@ -155,6 +126,5 @@
                 <origin xyz="0.0023249999999999668501 0.080077693916664902107 0.031949999999999985356" rpy="3.141592653589793116 -0 -3.141592653589793116" />
                 <geometry>
-                    <mesh filename="package://robot_description/meshes/shunk/visual/almofada.dae"/>
-                    <!--xacro:get_mesh name="almofada" type="visual"/-->
+                    <mesh filename="package://robot_description/meshes/schunk_egh80/visual/almofada.dae"/>
                 </geometry>
             </visual>
@@ -162,6 +132,5 @@
                 <origin xyz="0.0023249999999999668501 0.080077693916664902107 0.031949999999999985356" rpy="3.141592653589793116 -0 -3.141592653589793116" />
                 <geometry>
-                    <mesh filename="package://robot_description/meshes/shunk/collision/almofada.stl"/>
-                    <!--xacro:get_mesh name="almofada" type="collision"/-->
+                    <mesh filename="package://robot_description/meshes/schunk_egh80/collision/almofada.stl"/>
                 </geometry>
             </collision>
@@ -169,6 +138,5 @@
                 <origin xyz="0.0018250000000000266877 0.033299999999999760347 0.040700000000000027822" rpy="0 1.570796326794896558 0" />
                 <geometry>
-                    <mesh filename="package://robot_description/meshes/shunk/visual/falanginha.dae"/>
-                    <!--xacro:get_mesh name="falanginha" type="visual"/-->
+                    <mesh filename="package://robot_description/meshes/schunk_egh80/visual/falanginha.dae"/>
                 </geometry>
             </visual>
@@ -176,6 +144,5 @@
                 <origin xyz="0.0018250000000000266877 0.033299999999999760347 0.040700000000000027822" rpy="0 1.570796326794896558 0" />
                 <geometry>
-                    <mesh filename="package://robot_description/meshes/shunk/collision/falanginha.stl"/>
-                    <!--xacro:get_mesh name="falanginha" type="collision"/-->
+                    <mesh filename="package://robot_description/meshes/schunk_egh80/collision/falanginha.stl"/>
                 </geometry>
             </collision>
@@ -183,6 +150,5 @@
                 <origin xyz="0.0026249999999999372793 0.033299999999999760347 0.040700000000000013944" rpy="0 1.570796326794896336 0" />
                 <geometry>
-                    <mesh filename="package://robot_description/meshes/shunk/visual/falange.dae"/>
-                    <!--xacro:get_mesh name="falange" type="visual"/-->
+                    <mesh filename="package://robot_description/meshes/schunk_egh80/visual/falange.dae"/>
                 </geometry>
             </visual>
@@ -190,6 +156,5 @@
                 <origin xyz="0.0026249999999999372793 0.033299999999999760347 0.040700000000000013944" rpy="0 1.570796326794896336 0" />
                 <geometry>
-                    <mesh filename="package://robot_description/meshes/shunk/collision/falange.stl"/>
-                    <!--xacro:get_mesh name="falange" type="collision"/-->
+                    <mesh filename="package://robot_description/meshes/schunk_egh80/collision/falange.stl"/>
                 </geometry>
             </collision>
@@ -197,6 +162,5 @@
                 <origin xyz="0.0023249999999999707533 0.065299999999999677747 0.040700000000000013944" rpy="0 1.570796326794896558 0" />
                 <geometry>
-                    <mesh filename="package://robot_description/meshes/shunk/visual/falangeta.dae"/>
-                    <!--xacro:get_mesh name="falangeta" type="visual"/-->
+                    <mesh filename="package://robot_description/meshes/schunk_egh80/visual/falangeta.dae"/>
                 </geometry>
             </visual>
@@ -204,6 +168,5 @@
                 <origin xyz="0.0023249999999999707533 0.065299999999999677747 0.040700000000000013944" rpy="0 1.570796326794896558 0" />
                 <geometry>
-                    <mesh filename="package://robot_description/meshes/shunk/collision/falangeta.stl"/>
-                    <!--xacro:get_mesh name="falangeta" type="visual"/-->
+                    <mesh filename="package://robot_description/meshes/schunk_egh80/collision/falangeta.stl"/>
                 </geometry>
             </collision>
@@ -211,6 +174,5 @@
                 <origin xyz="0.0026250000000000014641 0.016000000000000000333 0.041500000000000002165" rpy="0 1.570796326794896558 0" />
                 <geometry>
-                    <mesh filename="package://robot_description/meshes/shunk/visual/guia_dedo.dae"/>
-                    <!--xacro:get_mesh name="guia_dedo" type="visual"/-->
+                    <mesh filename="package://robot_description/meshes/schunk_egh80/visual/guia_dedo.dae"/>
                 </geometry>
             </visual>
@@ -218,6 +180,5 @@
                 <origin xyz="0.0026250000000000014641 0.016000000000000000333 0.041500000000000002165" rpy="0 1.570796326794896558 0" />
                 <geometry>
-                    <mesh filename="package://robot_description/meshes/shunk/collision/guia_dedo.stl"/>
-                    <!--xacro:get_mesh name="guia_dedo" type="visual"/-->
+                    <mesh filename="package://robot_description/meshes/schunk_egh80/collision/guia_dedo.stl"/>
                 </geometry>
             </collision>
@@ -228,7 +189,7 @@
             </inertial>
         </link>
-        <joint name="${tf_prefix}gripper_base_joint" type="fixed">
+        <joint name="${prefix}gripper_base_joint" type="fixed">
             <origin xyz="0 0 0" rpy="0 0 1.570796326794896558" />
-            <parent link="${tf_prefix}tool0" />
+            <parent link="${prefix}tool0" />
             <child link="schunk_egh80_link" />
             <axis xyz="0 0 1"/>
@@ -237,5 +198,14 @@
         </joint>
         <!-- Juntas dos dedos -->
-        <joint name="${tf_prefix}dedo_esq_joint" type="prismatic">
+        <joint name="${prefix}dedo_dir_joint" type="prismatic">
+            <origin xyz="0.032500000000000028866 0.0036249999999999928113 0.10919999999999996376" rpy="1.570796326794896558 0 -1.570796326794896558" />
+            <axis xyz="0 0 1"/>
+            <limit effort="1" velocity="0.08" accelerarion="0.1" lower="0.0" upper="0.040"/>
+            <joint_properties friction="0.0"/>
+            <parent link="schunk_egh80_link" />
+            <child link="dedo_dir" />
+            <mimic joint="${prefix}dedo_esq_joint" multiplier="1" />
+        </joint>
+        <joint name="${prefix}dedo_esq_joint" type="prismatic">
             <origin xyz="-0.022499999999999978351 -0.0016250000000000075148 0.10919999999999994988" rpy="1.570796326794896558 0 1.570796326794896558" />
             <axis xyz="0 0 1" />
@@ -245,13 +215,4 @@
             <child link="dedo_esq"/>
         </joint>
-       <joint name="${tf_prefix}dedo_dir_joint" type="prismatic">
-            <origin xyz="0.032500000000000028866 0.0036249999999999928113 0.10919999999999996376" rpy="1.570796326794896558 0 -1.570796326794896558" />
-            <axis xyz="0 0 1"/>
-            <limit effort="1" velocity="0.08" accelerarion="0.1" lower="0.0" upper="0.040"/>
-            <joint_properties friction="0.0"/>
-            <parent link="schunk_egh80_link" />
-            <child link="dedo_dir" />
-            <mimic joint="${prefix}dedo_esq_joint" multiplier="-1" />
-        </joint>
     </xacro:macro>
 </robot>

File: src/robot_description/urdf/schunk_egh80/schunk_egh80_gripper.xacro (robot description, xacro)
@@ -34,6 +34,6 @@
     </inertial>
   </link>
-  <xacro:robotiq_85_gripper prefix="" parent="gripper_root_link" >
+  <xacro:schunk_egh80_gripper prefix="" parent="gripper_root_link" >
     <origin xyz="0.05 0 0.85" rpy="0 0 0"/>
-  </xacro:robotiq_85_gripper>
+  </xacro:schunk_egh80_gripper>
 </robot>
