Commit message: Add files via upload

File: src/ur3e_moveit_config/config/ur3e_egh80.urdf (robot description, URDF)
Before this commit: robot ur3e_egh80, 15 links, 14 joints
Links:
- link shoulder_link: mass 1.98 -> 3.7
Joints:
- joint shoulder_pan_joint: limit lower=-3.141592653589793 upper=3.141592653589793 effort=56.0 velocity=1.57079 -> lower=-3.141592653589793 upper=3.141592653589793 effort=56.0 velocity=3.15
